File: hardware-kicad/pcb/seedsigner-luckfox-pico/seedsigner-luckfox-devboard.kicad_sch (KiCad schematic)
At the start: 37 parts, among them J1 Conn_01x10, J2 Conn_01x05, U1 LuckFox_Pico, U2 RASPBERRY_PI_3_MODEL_B+

Commit message: auto-route and cleanup of pico mini devboard
Changed lines of the file:
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@@
-		)
-	)
-	(label "BACKLIGHT"
-		(at 25.4 55.88 180)
-		(effects
-			(font
-				(size 1.27 1.27)
-			)
-			(justify right bottom)
 		)
 	)
@@
 					(unit 1)
 				)
-			)
-		)
-	)
-	(symbol
-		(lib_id "power:+3.3V")
-		(at 27.94 53.34 0)
-		(unit 1)
-		(exclude_from_sim no)
-		(in_bom yes)
-		(on_board yes)
-		(dnp no)
-		(property "Reference" "#PWR012"
-			(at 27.94 57.15 0)
-			(effects
-				(font
-					(size 1.27 1.27)
-				)
-				(hide yes)
-			)
-		)
-		(property "Value" "+3.3V"
-			(at 27.94 48.26 0)
-			(effects
-				(font
-					(size 1.27 1.27)
-				)
-			)
-		)
-		(property "Footprint" ""
-			(at 27.94 53.34 0)
-			(effects
-				(font
-					(size 1.27 1.27)
-				)
-				(hide yes)
-			)
-		)
-		(property "Datasheet" ""
-			(at 27.94 53.34 0)
-			(effects
-				(font
-					(size 1.27 1.27)
-				)
-				(hide yes)
-			)
-		)
-		(property "Description" ""
-			(at 27.94 53.34 0)
-			(effects
-				(font
-					(size 1.27 1.27)
-				)
-				(hide yes)
-			)
-		)
-		(pin "1"
-		)
-		(instances
-			(project "seedsigner-luckfox-devboard"
-				(path "/dd9f0a7b-8b90-4e47-9769-d29b64af2c20"
-					(reference "#PWR012")
-					(unit 1)
-				)
