File: hardware-kicad/pcb/seedsigner-luckfox-pico-mini/seedsigner-luckfox-pico-mini.kicad_pcb (KiCad board)
At the start: 2 copper layers, 80 x 60 mm, 22 parts, among them U1 LuckFox_Pico_MINI, U2 RASPBERRY_PI_3_MODEL_B+

Commit message: cleanup project paths and make sure symbols and footprints are committed
Parts:
- U2: value RASPBERRY_PI_3_MODEL_B+ -> WAVESHARE_LCD_BUTTON_BOARD_1.3in
Connections:
- U2 pad 10: unconnected-(U2-RXD0/GPIO15-Pad10) -> (no net)
- U2 pad 11: unconnected-(U2-GPIO17/GPIO_GEN0-Pad11) -> (no net)
- U2 pad 12: unconnected-(U2-GPIO18/GPIO_GEN1-Pad12) -> (no net)
- U2 pad 15: unconnected-(U2-GPIO22/GPIO_GEN3-Pad15) -> (no net)
- U2 pad 16: unconnected-(U2-GPIO23/GPIO_GEN4-Pad16) -> (no net)
- U2 pad 21: unconnected-(U2-GPIO9/SPI_MISO-Pad21) -> (no net)
- U2 pad 26: unconnected-(U2-GPIO7/~{SPI_CE1}-Pad26) -> (no net)
- U2 pad 27: unconnected-(U2-ID_SD-Pad27) -> (no net)
- U2 pad 28: unconnected-(U2-ID_SC-Pad28) -> (no net)
- U2 pad 3: unconnected-(U2-GPIO2/SDA1-Pad3) -> (no net)
- U2 pad 32: unconnected-(U2-GPIO12-Pad32) -> (no net)
- U2 pad 5: unconnected-(U2-GPIO3/SCL1-Pad5) -> (no net)
- U2 pad 7: unconnected-(U2-GPIO4/GPIO_GCKL-Pad7) -> (no net)
- U2 pad 8: unconnected-(U2-TXD0/GPIO14-Pad8) -> (no net)
