File: hardware-kicad/pcb/seedsigner-luckfox-shipit/modules.kicad_sch (KiCad schematic)
At the start: 3 parts, among them U1 LuckFox_Pico_MINI, U2 LuckFox_Pico_PLUS_PRO

Commit message: 2 different pcbs almost done
Parts:
- removed U1: LuckFox_Pico_MINI, seedsigner-luckfox:LUCKFOX_PICO_MINI, symbol Luckfox:LuckFox_Pico_MINI
- added R10, R11, R12, R13, R14, R9: 10K, Resistor_SMD:R_0805_2012Metric_Pad1.20x1.40mm_HandSolder, symbol Device:R
- added U2: PCA9539PW_112, seedsigner-luckfox:SOP65P640X110-24N, symbol SeedSigner:PCA9539PW_112
- U1: renamed from U2; footprint (none) -> seedsigner-luckfox:LUCKFOX_PICO
Connections:
- net DC is gone; now on net LCD_DC: LCD1.3 (DC)
- net RST is gone; now on net LCD_RST: LCD1.2 (RST)
- net +3.3V: now also U1.36 (3V3(OUT)), R10.1, R11.1, R12.1, R13.1, R14.1, R9.1, U2.24 (VDD)
- net BACKLIGHT_PWM: now also U1.17 (GPIO2_B0_d)
- net GND: now also U1.38 (GND), U2.12 (VSS)
- net JOYSTICK_DOWN: now also U1.6 (UART4_TX_M1/GPIO1_C5_d), U2.8 (IO0_4)
- net JOYSTICK_LEFT: now also U1.10 (GPIO1_D3_d), U2.11 (IO0_7)
- net JOYSTICK_PRESS: now also U1.7 (UART4_RX_M1/GPIO1_C4_d), U2.9 (IO0_5)
- net JOYSTICK_RIGHT: now also U1.5 (UART4_RTS_M1/GPIO1_C6_d), U2.7 (IO0_3)
- net JOYSTICK_UP: now also U1.9 (GPIO1_D4_d), U2.10 (IO0_6)
- net KEY1: now also U1.4 (UART4_CTS_M1/GPIO1_C7_d), U2.6 (IO0_2)
- net KEY2: now also U1.2 (UART2_RX_M1/GPIO1_B3_d), U2.5 (IO0_1)
- net KEY3: now also U1.1 (UART2_TX_M1/GPIO1_B2_d), U2.4 (IO0_0)
- net SPI_CS: now also U1.12 (GPIO2_C0_d)
- net SPI_MOSI: now also U1.15 (GPIO1_C2_d)
- net SPI_SCLK: now also U1.14 (GPIO1_C1_d)
- net LCD_DC: now reaches U1.19 (GPIO1_D0_d)
- net LCD_RST: now reaches U1.20 (GPIO1_D1_d)
- net IO_INT: now reaches U1.22 (GPIO2_A5_d)
- net IO_INT: now also R14.2, U2.1 (~INT)
- net I2C_SDA: now reaches U1.24 (GPIO2_D0_d)
- net I2C_SDA: now also R10.2, U2.23 (SDA)
- net I2C_SCL: now reaches U1.25 (GPIO2_A1_d)
- net I2C_SCL: now also R9.2, U2.22 (SCL)
- net VSYS: now reaches U1.39 (VSYS)
- net VBUS: now reaches U1.40 (VBUS)
- new net: R13.2, U2.2 (A1)
- new net: R12.2, U2.21 (A0)
- new net: R11.2, U2.3 (~RESET)
Other:
- moved on the sheet: U1

Commit message: pcb checkin, ordered
Parts:
- added C1: 100nF, Capacitor_SMD:C_0805_2012Metric_Pad1.18x1.45mm_HandSolder, symbol Device:C
Connections:
- net +3.3V: now also C1.1
- net GND: now also C1.2
Changed lines of the file:
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@@
+	)
+	(symbol
+		(lib_id "power:+3.3V")
+		(at 113.03 139.7 0)
+		(unit 1)
+		(exclude_from_sim no)
+		(in_bom yes)
+		(on_board yes)
+		(dnp no)
+		(fields_autoplaced yes)
+		(property "Reference" "#PWR014"
+			(at 113.03 143.51 0)
+			(effects
+				(font
+					(size 1.27 1.27)
+				)
+				(hide yes)
+			)
+		)
+		(property "Value" "+3.3V"
+			(at 113.03 134.62 0)
+			(effects
+				(font
+					(size 1.27 1.27)
+				)
+			)
+		)
+		(property "Footprint" ""
+			(at 113.03 139.7 0)
+			(effects
+				(font
+					(size 1.27 1.27)
+				)
+				(hide yes)
+			)
+		)
+		(property "Datasheet" ""
+			(at 113.03 139.7 0)
+			(effects
+				(font
+					(size 1.27 1.27)
+				)
+				(hide yes)
+			)
+		)
+		(property "Description" ""
+			(at 113.03 139.7 0)
+			(effects
+				(font
+					(size 1.27 1.27)
+				)
+				(hide yes)
+			)
+		)
+		(pin "1"
+		)
+		(instances
+			(project "seedsigner-luckfox-shipit"
+				(path "/cdb42d61-6e7c-45da-bb95-2df00473b6b5/83443f2e-49ec-4a5d-8e70-32df6acdc6b1"
+					(reference "#PWR014")
+					(unit 1)
+				)
+			)
+		)
 	)
 	(symbol
@@
 	)
 	(symbol
+		(lib_id "power:GND")
+		(at 113.03 147.32 0)
+		(unit 1)
+		(exclude_from_sim no)
+		(in_bom yes)
+		(on_board yes)
+		(dnp no)
+		(fields_autoplaced yes)
+		(property "Reference" "#PWR015"
+			(at 113.03 153.67 0)
+			(effects
+				(font
+					(size 1.27 1.27)
+				)
+				(hide yes)
+			)
+		)
+		(property "Value" "GND"
+			(at 113.03 152.4 0)
+			(effects
+				(font
+					(size 1.27 1.27)
+				)
+			)
+		)
+		(property "Footprint" ""
+			(at 113.03 147.32 0)
+			(effects
+				(font
+					(size 1.27 1.27)
+				)
+				(hide yes)
+			)
+		)
+		(property "Datasheet" ""
+			(at 113.03 147.32 0)
+			(effects
+				(font
+					(size 1.27 1.27)
+				)
+				(hide yes)
+			)
+		)
+		(property "Description" ""
+			(at 113.03 147.32 0)
+			(effects
+				(font
+					(size 1.27 1.27)
+				)
+				(hide yes)
+			)
+		)
+		(pin "1"
+		)
+		(instances
+			(project "seedsigner-luckfox-shipit"
+				(path "/cdb42d61-6e7c-45da-bb95-2df00473b6b5/83443f2e-49ec-4a5d-8e70-32df6acdc6b1"
+					(reference "#PWR015")
+					(unit 1)
+				)
+			)
+		)
+	)
+	(symbol
 		(lib_id "power:+3.3V")
 		(at 69.85 82.55 90)
@@
 					(unit 1)
 				)
+			)
+		)
+	)
+	(symbol
+		(lib_id "Device:C")
+		(at 113.03 143.51 0)
+		(unit 1)
+		(exclude_from_sim no)
+		(in_bom yes)
+		(on_board yes)
+		(dnp no)
+		(fields_autoplaced yes)
+		(property "Reference" "C1"
+			(at 116.84 142.2399 0)
+			(effects
+				(font
+					(size 1.27 1.27)
+				)
+				(justify left)
+			)
+		)
+		(property "Value" "100nF"
+			(at 116.84 144.7799 0)
+			(effects
+				(font
+					(size 1.27 1.27)
+				)
+				(justify left)
+			)
+		)
+		(property "Footprint" "Capacitor_SMD:C_0805_2012Metric_Pad1.18x1.45mm_HandSolder"
+			(at 113.9952 147.32 0)
+			(effects
+				(font
+					(size 1.27 1.27)
+				)
+				(hide yes)
+			)
+		)
+		(property "Datasheet" "~"
+			(at 113.03 143.51 0)
+			(effects
+				(font
+					(size 1.27 1.27)
+				)
+				(hide yes)
+			)
+		)
+		(property "Description" "Unpolarized capacitor"
+			(at 113.03 143.51 0)
+			(effects
+				(font
+					(size 1.27 1.27)
+				)
+				(hide yes)
+			)
+		)
+		(pin "1"
+		)
+		(pin "2"
+		)
+		(instances
+			(project ""
+				(path "/cdb42d61-6e7c-45da-bb95-2df00473b6b5/83443f2e-49ec-4a5d-8e70-32df6acdc6b1"
+					(reference "C1")
+					(unit 1)
+				)
