File: hardware-kicad/pcb/seedsigner-luckfox-shipit/seedsigner-luckfox-shipit.kicad_pcb (KiCad board)
At the start: 2 copper layers, 70 x 80 mm, 25 parts, among them SW1 SW_Push, SW2 SW_Push, SW3 SW_Push, SW4 SW_Push, SW5 SW_Push, SW6 SW_Push, SW7 SW_Push, SW8 SW_Push, U1 LuckFox_Pico_MINI

Commit message: 2 different pcbs almost done
Parts:
- added R10: 10K, Resistor_SMD:R_0805_2012Metric_Pad1.20x1.40mm_HandSolder, F.Cu at (26.0, 4.00)
- added R11: 10K, Resistor_SMD:R_0805_2012Metric_Pad1.20x1.40mm_HandSolder, F.Cu at (6.00, 39.0)
- added R12: 10K, Resistor_SMD:R_0805_2012Metric_Pad1.20x1.40mm_HandSolder, F.Cu at (8.00, 39.0)
- added R13: 10K, Resistor_SMD:R_0805_2012Metric_Pad1.20x1.40mm_HandSolder, F.Cu at (4.00, 39.0)
- added R14: 10K, Resistor_SMD:R_0805_2012Metric_Pad1.20x1.40mm_HandSolder, F.Cu at (10.0, 4.00)
- added R9: 10K, Resistor_SMD:R_0805_2012Metric_Pad1.20x1.40mm_HandSolder, F.Cu at (28.0, 4.00)
- added TP1: TestPoint, seedsigner-luckfox:TestPoint_Pad_1.5x1.5mm, F.Cu at (53.0, 4.00)
- added TP2: TestPoint, seedsigner-luckfox:TestPoint_Pad_1.5x1.5mm, F.Cu at (49.0, 4.00)
- added TP3: TestPoint, seedsigner-luckfox:TestPoint_Pad_1.5x1.5mm, F.Cu at (40.0, 4.00)
- added TP4: TestPoint, seedsigner-luckfox:TestPoint_Pad_1.5x1.5mm, F.Cu at (45.0, 4.00)
- added U2: PCA9539PW_112, seedsigner-luckfox:SOP65P640X110-24N, F.Cu at (7.00, 45.0)
- U1: value LuckFox_Pico_MINI -> LuckFox_Pico_PLUS_PRO; footprint seedsigner-luckfox:LUCKFOX_PICO_MINI -> seedsigner-luckfox:LUCKFOX_PICO
- moved LOGO2 68.8 mm to (35.0, 18.0)
- moved ART1 56.3 mm to (66.0, 27.0), turned to 90 degrees
- moved U1 43.4 mm to (56.0, 27.0), turned to 90 degrees
- moved LOGO1 39.8 mm to (66.0, 55.0), turned to 90 degrees
- moved H3 10.0 mm to (67.0, 67.0)
- moved H4 10.0 mm to (3.00, 67.0)
- moved R4 6.00 mm to (13.0, 38.0)
- moved SW1 6.00 mm to (49.0, 47.0)
- moved SW2 6.00 mm to (49.0, 56.0)
- moved SW3 6.00 mm to (49.0, 65.0)
- moved SW4 6.00 mm to (8.00, 56.0)
- moved R1 6.00 mm to (44.0, 38.0)
- moved R2 6.00 mm to (47.0, 38.0)
- moved R3 6.00 mm to (50.0, 38.0)
- moved R5 6.00 mm to (19.0, 38.0)
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Connections:
- LCD1 pad 1: /Modules/BACKLIGHT_PWM -> BACKLIGHT_PWM
- LCD1 pad 2: /Modules/RST -> LCD_RST
- LCD1 pad 3: /Modules/DC -> LCD_DC
- LCD1 pad 4: /Modules/SPI_CS -> SPI_CS
- LCD1 pad 5: /Modules/SPI_SCLK -> SPI_SCLK
- LCD1 pad 6: /Modules/SPI_MOSI -> SPI_MOSI
- U1 pad 1: unconnected-(U1-VBUS-Pad1) -> KEY3
- U1 pad 10: /Modules/DC -> JOYSTICK_LEFT
- U1 pad 11: KEY3 -> unconnected-(U1-GPIO2_B1_d-Pad11)
- U1 pad 12: JOYSTICK_LEFT -> SPI_CS
- U1 pad 13: JOYSTICK_UP -> unconnected-(U1-GND-Pad13)
- U1 pad 14: JOYSTICK_PRESS -> SPI_SCLK
- U1 pad 15: JOYSTICK_DOWN -> SPI_MOSI
- U1 pad 16: JOYSTICK_RIGHT -> unconnected-(U1-GPIO1_C3_d-Pad16)
- U1 pad 17: KEY1 -> BACKLIGHT_PWM
- U1 pad 18: /Modules/BACKLIGHT_PWM -> unconnected-(U1-GND-Pad18)
- U1 pad 19: unconnected-(U1-GPIO4_C0_z-Pad19) -> LCD_DC
- U1 pad 2: GND -> KEY2
- U1 pad 20: unconnected-(U1-GPIO4_C1_z-Pad20) -> LCD_RST
- U1 pad 21: GND -> unconnected-(U1-GPIO2_A4_d-Pad21)
- U1 pad 22: unconnected-(U1-1V8(OUT)-Pad22) -> IO_INT
- U1 pad 3: +3.3V -> unconnected-(U1-GND-Pad3)
- U1 pad 4: unconnected-(U1-GPIO1_B2_d-Pad4) -> KEY1
- U1 pad 5: KEY2 -> JOYSTICK_RIGHT
- U1 pad 6: /Modules/SPI_CS -> JOYSTICK_DOWN
- U1 pad 7: /Modules/SPI_SCLK -> JOYSTICK_PRESS
- U1 pad 8: /Modules/SPI_MOSI -> unconnected-(U1-GND-Pad8)
- U1 pad 9: /Modules/RST -> JOYSTICK_UP
Routing:
- net +3.3V: track 137.3 -> 205.5 mm, vias 2 -> 6
- net BACKLIGHT_PWM: track 0.00 -> 61.4 mm, vias 0 -> 1
- net LCD_RST: track 0.00 -> 60.4 mm
- net LCD_DC: track 0.00 -> 56.8 mm
- net /Modules/BACKLIGHT_PWM: track 52.6 -> 0.00 mm, vias 1 -> 0
- net I2C_SDA: track 0.00 -> 49.6 mm, vias 0 -> 2
- net I2C_SCL: track 0.00 -> 49.3 mm
- net /Modules/SPI_CS: track 47.3 -> 0.00 mm, vias 1 -> 0
- net /Modules/SPI_SCLK: track 47.1 -> 0.00 mm, vias 1 -> 0
- net SPI_MOSI: track 0.00 -> 45.7 mm
- net IO_INT: track 0.00 -> 44.9 mm
- net SPI_CS: track 0.00 -> 42.6 mm, vias 0 -> 1
- net SPI_SCLK: track 0.00 -> 42.0 mm
- net /Modules/SPI_MOSI: track 37.8 -> 0.00 mm, vias 1 -> 0
- net JOYSTICK_RIGHT: track 55.2 -> 91.6 mm, vias 0 -> 3
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Other:
- board size 70 x 80 mm -> 70 x 70 mm
- board text added: "07/03/2025"
- board text added: "BL"
- board text added: "CS"
- board text added: "DC"
- board text added: "GND"
- board text added: "LuckFox Big Screen"
- board text added: "MOSI"
- board text added: "RST"
- board text added: "SCLK"
- board text added: "VCC"
- board text removed: "TODO: Rotate screen so connector is on the right"

Commit message: pcb checkin, ordered
Parts:
- added C1: 100nF, Capacitor_SMD:C_0805_2012Metric_Pad1.18x1.45mm_HandSolder, F.Cu at (12.0, 46.0)
Routing:
- net +3.3V: track 205.5 -> 204.4 mm
