File: hardware-kicad/pcb/seedsigner-hardware-dev-v1/ArtAndSymbols.kicad_sch (KiCad schematic)
At the start: 3 parts

Commit message: close to ordering on jlcpcb
Parts:
- ART1, LOGO2: now left out of the parts list
Changed lines of the file:
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@@
 		(unit 1)
 		(exclude_from_sim no)
-		(in_bom yes)
+		(in_bom no)
 		(on_board yes)
 		(dnp no)
@@
 		(unit 1)
 		(exclude_from_sim no)
-		(in_bom yes)
+		(in_bom no)
 		(on_board yes)
 		(dnp no)

Commit message: pcb checkin, ordered
Parts:
- added ART2: Modulo, seedsigner-luckfox:modulo-1, symbol seedsigner:LIGHTNINGSPORE
Changed lines of the file:
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@@
+	(symbol
+		(lib_id "seedsigner:LIGHTNINGSPORE")
+		(at 95.25 91.44 0)
+		(unit 1)
+		(exclude_from_sim no)
+		(in_bom no)
+		(on_board yes)
+		(dnp no)
+		(fields_autoplaced yes)
+		(property "Reference" "ART2"
+			(at 100.33 90.8049 0)
+			(effects
+				(font
+					(size 1.27 1.27)
+				)
+				(justify left)
+			)
+		)
+		(property "Value" "Modulo"
+			(at 100.33 92.71 0)
+			(effects
+				(font
+					(size 1.27 1.27)
+				)
+				(justify left)
+			)
+		)
+		(property "Footprint" "seedsigner-luckfox:modulo-1"
+			(at 95.25 91.44 0)
+			(effects
+				(font
+					(size 1.27 1.27)
+				)
+				(hide yes)
+			)
+		)
+		(property "Datasheet" ""
+			(at 95.25 91.44 0)
+			(effects
+				(font
+					(size 1.27 1.27)
+				)
+				(hide yes)
+			)
+		)
+		(property "Description" ""
+			(at 95.25 91.44 0)
+			(effects
+				(font
+					(size 1.27 1.27)
+				)
+				(hide yes)
+			)
+		)
+		(instances
+			(project "seedsigner-hardware-dev-v1"
+				(path "/80ddcc25-987b-44b8-ab4f-432d39ad0241/5cb8505d-b540-42ed-b4a9-9676439affb7"
+					(reference "ART2")
+					(unit 1)
+				)
+			)
+		)
+	)
 	(symbol
 		(lib_id "seedsigner:LIGHTNINGSPORE")
