File: hardware-kicad/pcb/seedsigner-hardware-dev-v1/seedsigner-hardware-dev-v1.kicad_sch (KiCad schematic)
At the start: 6 parts, among them J1 Conn_01x08_MountingPin

Commit message: 2 different pcbs almost done
Parts:
- removed J1: Conn_01x08_MountingPin, Connector_PinHeader_2.54mm:PinHeader_1x08_P2.54mm_Horizontal, symbol Connector_Generic_MountingPin:Conn_01x08_MountingPin
- added LCD2: ST7789, Connector_PinHeader_2.54mm:PinHeader_1x08_P2.54mm_Vertical, symbol SeedSigner:LCD_ST7789
- added TP5, TP6: TestPoint, TestPoint:TestPoint_Pad_D1.0mm, symbol Connector:TestPoint
- H1, H2, H3, H4: now left out of the parts list
Connections:
- net +3.3V: now also LCD2.8 (VCC), TP6.1
- net GND: now also LCD2.7 (GND), TP5.1
- net SPI_CS: now also LCD2.4 (SPI_CS)
- net SPI_MOSI: now also LCD2.6 (SPI_MOSI)
- net SPI_SCLK: now also LCD2.5 (SPI_SCLK)
- net BACKLIGHT renamed BACKLIGHT_PWM
- net BACKLIGHT_PWM: now also LCD2.1 (BL)
- net DC renamed LCD_DC
- net LCD_DC: now also LCD2.3 (DC)
- net RST renamed LCD_RST
- net LCD_RST: now also LCD2.2 (RST)

Commit message: pcb checkin, ordered
Parts:
- added J1: Conn_01x04, Connector:NS-Tech_Grove_1x04_P2mm_Vertical, symbol Connector_Generic:Conn_01x04
- added TP10, TP7, TP8, TP9: TestPoint, TestPoint:TestPoint_Pad_D1.0mm, symbol Connector:TestPoint
Connections:
- net +3.3V: now also J1.3 (Pin_3), TP10.1, TP8.1
- net GND: now also J1.4 (Pin_4), TP7.1, TP9.1
- new net I2C_SCL: J1.1 (Pin_1)
- new net I2C_SDA: J1.2 (Pin_2)
